Commit message: tray feature

File: robot_description/urdf/robot.gazebo.xacro (robot description, xacro)
@@ -15,5 +15,5 @@
     <transmission name="tran1">
         <type>transmission_interface/SimpleTransmission</type>
-        <joint name="joint_lifting_tray">
+        <joint name="joint_piston">
             <hardwareInterface>hardware_interface/EffortJointInterface</hardwareInterface>
         </joint>
@@ -23,4 +23,19 @@
         </actuator>
     </transmission>
+    <!-- <transmission name="tran2">
+        <type>transmission_interface/SimpleTransmission</type>
+        <joint name="joint_tray">
+            <hardwareInterface>hardware_interface/EffortJointInterface</hardwareInterface>
+        </joint>
+        <actuator name="motor2">
+            <hardwareInterface>hardware_interface/EffortJointInterface</hardwareInterface>
+            <mechanicalReduction>1</mechanicalReduction>
+        </actuator>
+    </transmission> -->
+    <gazebo>
+        <plugin name="joint_state_publisher" filename="libgazebo_ros_joint_state_publisher.so">
+            <jointName>joint_piston, joint_tray</jointName>
+        </plugin>
+    </gazebo>
     <gazebo>
         <plugin name="gazebo_ros_control" filename="libgazebo_ros_control.so">

File: robot_description/urdf/robot.urdf.xacro (robot description, xacro)
@@ -12,10 +12,16 @@
     <origin rpy="0 0 -1.57" xyz="-0.0005 -0.23 0.109"/>
   </joint>
-  <joint name="joint_lifting_tray" type="prismatic">
-    <parent link="carcaca"/>
-    <child link="lifting_tray"/>
+  <joint name="joint_piston" type="prismatic">
+    <parent link="carcaca"/>
+    <child link="piston"/>
     <origin rpy="0 0 0" xyz="0 0 0.1318"/>
     <axis xyz="0 0 1"/>
-    <limit effort="100" lower="0" upper="0.04" velocity="1"/>
+    <limit effort="10" lower="0" upper="0.04" velocity="0.1"/>
+  </joint>
+  <joint name="joint_tray" type="continuous">
+    <parent link="piston"/>
+    <child link="tray"/>
+    <origin rpy="0 0 0" xyz="0 0 0"/>
+    <axis xyz="0 0 1"/>
   </joint>
   <joint name="joint_wheel_front_right" type="fixed">
@@ -188,5 +194,5 @@
     </visual>
   </link>
-  <gazebo reference="lifting_tray">
+  <gazebo reference="piston">
     <selfCollide>true</selfCollide>
     <mu1 value="0.1"/>
@@ -196,20 +202,47 @@
     <fdir1 value="0 0 0"/>
   </gazebo>
-  <link name="lifting_tray">
-    <inertial>
-      <mass value="0.5"/>
+  <link name="piston">
+    <inertial>
+      <mass value="0.1"/>
       <origin rpy="0  0  0" xyz="0 0 0"/>
       <inertia ixx="1" ixy="0" ixz="0" iyy="1" iyz="0" izz="1"/>
     </inertial>
-    <collision name="lifting_tray_collision">
+    <collision name="piston_collision">
       <origin rpy="0  0  0" xyz="0 0 0"/>
       <geometry>
-        <mesh filename="package://robot_description/models/laser_robot/meshes/lifting.dae" scale="1 1 1"/>
-      </geometry>
-    </collision>
-    <visual name="lifting_tray_visual">
+        <mesh filename="package://robot_description/models/laser_robot/meshes/piston.dae" scale="1 1 1"/>
+      </geometry>
+    </collision>
+    <visual name="piston_visual">
       <origin rpy="0  0  0" xyz="0 0 0"/>
       <geometry>
-        <mesh filename="package://robot_description/models/laser_robot/meshes/lifting.dae" scale="1 1 1"/>
+        <mesh filename="package://robot_description/models/laser_robot/meshes/piston.dae" scale="1 1 1"/>
+      </geometry>
+    </visual>
+  </link>
+  <gazebo reference="tray">
+    <selfCollide>true</selfCollide>
+    <mu1 value="0.09"/>
+    <mu2 value="0.09"/>
+    <kp value="10000000.0" />
+    <kd value="10000" />
+    <fdir1 value="0 0 0"/>
+  </gazebo>
+  <link name="tray">
+    <inertial>
+      <mass value="0.01"/>
+      <origin rpy="0 0 0" xyz="0 0 0"/>
+      <inertia ixx="1" ixy="0.0" ixz="0.0" iyy="1" iyz="0.0" izz="1"/>
+    </inertial>
+    <collision name="tray_collision">
+      <origin rpy="0 0 0" xyz="0 0 0"/>
+      <geometry>
+        <mesh filename="package://robot_description/models/laser_robot/meshes/tray.dae" scale="1 1 1"/>
+      </geometry>
+    </collision>
+    <visual name="tray_visual">
+      <origin rpy="0 0 0" xyz="0 0 0"/>
+      <geometry>
+        <mesh filename="package://robot_description/models/laser_robot/meshes/tray.dae" scale="1 1 1"/>
       </geometry>
     </visual>

Commit message: Add RPLidar

File: robot_description/urdf/robot.gazebo.xacro (robot description, xacro)
@@ -1,5 +1,4 @@
 <?xml version="1.0" ?>
 <robot xmlns:xacro="http://www.ros.org/wiki/xacro">
-  <xacro:arg name="camera_1_visual" default="false"/>
     <xacro:macro name="omni_steering" params="">
         <gazebo>
@@ -89,4 +88,5 @@
         </plugin>
     </gazebo>
+    <xacro:arg name="camera_1_visual" default="false"/>
     <gazebo reference="camera_1">
         <sensor type="camera" name="camera1">
@@ -126,21 +126,21 @@
         </sensor>
     </gazebo>
-  <gazebo reference="lidar">
+  <gazebo reference="rplidar">
     <sensor type="ray" name="laser_sensor">
       <pose>0 0 0 0 0 0</pose>
-      <visualize>false</visualize>
-      <update_rate>40</update_rate>
+      <visualize>true</visualize>
+      <update_rate>20</update_rate>
       <ray>
         <scan>
           <horizontal>
-            <samples>720</samples>
+            <samples>${14400/20}</samples>
             <resolution>1</resolution>
-            <min_angle>-1.1775</min_angle>
-            <max_angle>1.1775</max_angle>
+            <min_angle>-3.14159265359</min_angle>
+            <max_angle>3.14159265359</max_angle>
           </horizontal>
         </scan>
         <range>
-          <min>0.10</min>
-          <max>10.0</max>
+          <min>0.15</min>
+          <max>14.0</max>
           <resolution>0.01</resolution>
         </range>
@@ -157,5 +157,5 @@
       <plugin name="gazebo_ros_head_hokuyo_controller" filename="libgazebo_ros_laser.so">
         <topicName>/my_robot/laser/scan</topicName>
-        <frameName>lidar</frameName>
+        <frameName>rplidar</frameName>
       </plugin>
     </sensor>

File: robot_description/urdf/robot.urdf.xacro (robot description, xacro)
@@ -12,4 +12,9 @@
     <origin rpy="0 0 -1.57" xyz="-0.0005 -0.23 0.109"/>
   </joint>
+  <joint name="joint_rplidar" type="fixed">
+    <parent link="carcaca"/>
+    <child link="rplidar"/>
+    <origin rpy="0 0 0" xyz="0.14 -0.17 0.27"/>
+  </joint>
   <joint name="joint_piston" type="prismatic">
     <parent link="carcaca"/>
@@ -17,5 +22,5 @@
     <origin rpy="0 0 0" xyz="0 0 0.1318"/>
     <axis xyz="0 0 1"/>
-    <limit effort="10" lower="0" upper="0.04" velocity="0.1"/>
+    <limit effort="0" lower="0" upper="0.04" velocity="0"/>
   </joint>
   <joint name="joint_tray" type="continuous">
@@ -195,5 +200,5 @@
   </link>
   <gazebo reference="piston">
-    <selfCollide>true</selfCollide>
+    <selfCollide>false</selfCollide>
     <mu1 value="0.1"/>
     <mu2 value="0.1"/>
@@ -204,7 +209,7 @@
   <link name="piston">
     <inertial>
-      <mass value="0.1"/>
+      <mass value="0.3"/>
       <origin rpy="0  0  0" xyz="0 0 0"/>
-      <inertia ixx="1" ixy="0" ixz="0" iyy="1" iyz="0" izz="1"/>
+      <inertia ixx="0" ixy="0" ixz="0" iyy="0" iyz="0" izz="0"/>
     </inertial>
     <collision name="piston_collision">
@@ -222,7 +227,7 @@
   </link>
   <gazebo reference="tray">
-    <selfCollide>true</selfCollide>
-    <mu1 value="0.09"/>
-    <mu2 value="0.09"/>
+    <selfCollide>false</selfCollide>
+    <mu1 value="0.1"/>
+    <mu2 value="0.1"/>
     <kp value="10000000.0" />
     <kd value="10000" />
@@ -231,7 +236,7 @@
   <link name="tray">
     <inertial>
-      <mass value="0.01"/>
-      <origin rpy="0 0 0" xyz="0 0 0"/>
-      <inertia ixx="1" ixy="0.0" ixz="0.0" iyy="1" iyz="0.0" izz="1"/>
+      <mass value="0.5"/>
+      <origin rpy="0 0 0" xyz="0 0 0"/>
+      <inertia ixx="0" ixy="0.0" ixz="0.0" iyy="0" iyz="0.0" izz="0"/>
     </inertial>
     <collision name="tray_collision">
@@ -340,3 +345,22 @@
     </visual>
   </link>
+  <link name="rplidar">
+    <inertial>
+      <mass value="0.1"/>
+      <origin rpy="0 0 0" xyz="0 0 0"/>
+      <inertia ixx="1" ixy="0" ixz="0" iyy="1" iyz="0" izz="1"/>
+    </inertial>
+    <collision name="rplidar_collision">
+      <origin rpy="0 0 1.20" xyz="-0.03 0.02 -0.02"/>
+      <geometry>
+        <mesh filename="package://robot_description/models/laser_robot/meshes/rplidar.dae" scale="0.7 0.7 0.7"/>
+      </geometry>
+    </collision>
+    <visual name="rplidar_visual">
+      <origin rpy="0 0 1.20" xyz="-0.03 0.02 -0.02"/>
+      <geometry>
+        <mesh filename="package://robot_description/models/laser_robot/meshes/rplidar.dae" scale="0.7 0.7 0.7"/>
+      </geometry>
+    </visual>
+  </link>
 </robot>
