Commit message: adjusting urdf

File: robot_description/urdf/robot.urdf.xacro (robot description, xacro)
@@ -1,366 +1,32 @@
-<?xml version="1.0" ?>
+<?xml version="1.0"?>
 <robot name="my_robot" xmlns:xacro="http://www.ros.org/wiki/xacro">
+  <!--=========================== PLUGINS ===========================-->
   <xacro:include filename="$(find robot_description)/urdf/robot.gazebo.xacro" />
-  <joint name="joint_camera_1" type="fixed">
-    <parent link="carcaca"/>
-    <child link="camera_1"/>
-    <origin rpy="0 1.57 0" xyz="0 -0.127 0.0367"/>
-  </joint>
-  <joint name="joint_lidar" type="fixed">
-    <parent link="carcaca"/>
-    <child link="lidar"/>
-    <origin rpy="0 0 -1.57" xyz="-0.0005 -0.23 0.109"/>
-  </joint>
-  <joint name="joint_rplidar" type="fixed">
-    <parent link="carcaca"/>
-    <child link="rplidar"/>
-    <origin rpy="0 0 0" xyz="0.14 -0.17 0.27"/>
-  </joint>
-  <joint name="joint_piston" type="prismatic">
-    <parent link="carcaca"/>
-    <child link="piston"/>
-    <origin rpy="0 0 0" xyz="0 0 0.1318"/>
-    <axis xyz="0 0 1"/>
-    <limit effort="0" lower="0" upper="0.04" velocity="0"/>
-  </joint>
-  <joint name="joint_tray" type="continuous">
-    <parent link="piston"/>
-    <child link="tray"/>
-    <origin rpy="0 0 0" xyz="0 0 0"/>
-    <axis xyz="0 0 1"/>
-  </joint>
-  <joint name="joint_wheel_front_right" type="fixed">
-    <parent link="carcaca"/>
-    <child link="wheel_front_right"/>
-    <origin rpy="0 1.57 0" xyz="0.193 -0.176 0.0508"/>
-  </joint>
-  <joint name="joint_wheel_rear_right" type="fixed">
-    <parent link="carcaca"/>
-    <child link="wheel_rear_right"/>
-    <origin rpy="0 1.57 0" xyz="0.193 0.176 0.0508"/>
-  </joint>
-  <joint name="joint_wheel_front_left" type="fixed">
-    <parent link="carcaca"/>
-    <child link="wheel_front_left"/>
-    <origin rpy="0 1.57 0" xyz="-0.214 -0.176 0.0508"/>
-  </joint>
-  <joint name="joint_wheel_rear_left" type="fixed">
-    <parent link="carcaca"/>
-    <child link="wheel_rear_left"/>
-    <origin rpy="0 1.57 0" xyz="-0.214 0.176 0.0508"/>
-  </joint>
-  <joint name="joint_right_wheel" type="revolute">
-    <parent link="carcaca"/>
-    <child link="right_wheel"/>
-    <origin rpy="0 1.57 0" xyz="0.193 0 0.0507"/>
-    <axis xyz="0 0 1"/>
-    <limit effort="-1.0" lower="-1e+16" upper="1e+16" velocity="-1.0"/>
-  </joint>
-  <joint name="joint_left_wheel" type="revolute">
-    <parent link="carcaca"/>
-    <child link="left_wheel"/>
-    <origin rpy="0 1.57 0" xyz="-0.214 0 0.0507"/>
-    <axis xyz="0 0 1"/>
-    <limit effort="-1.0" lower="-1e+16" upper="1e+16" velocity="-1.0"/>
-  </joint>
-  <gazebo reference="carcaca">
-    <selfCollide>true</selfCollide>
-    <mu1 value="0.3"/>
-    <mu2 value="0.3"/>
-    <kp value="10000000.0" />
-    <kd value="1000" />
-    <fdir1 value="0 0 0"/>
-  </gazebo>
-  <link name="carcaca">
-    <inertial>
-      <mass value="15"/>
-      <origin rpy="0  0  3.14" xyz="0  0  0.0118"/>
-      <inertia ixx="1" ixy="0" ixz="0" iyy="1" iyz="0" izz="1"/>
-    </inertial>
-    <collision name="carcaca_collision">
-      <origin rpy="0  0  3.14" xyz="0  0  0.0118"/>
-      <geometry>
-        <mesh filename="package://robot_description/models/laser_robot/meshes/carcaca.dae" scale="1 1 1"/>
-      </geometry>
-    </collision>
-    <visual name="carcaca_visual">
-      <origin rpy="0  0  3.14" xyz="0  0  0.0118"/>
-      <geometry>
-        <mesh filename="package://robot_description/models/laser_robot/meshes/carcaca.dae" scale="1 1 1"/>
-      </geometry>
-    </visual>
-  </link>
-  <gazebo reference="wheel_front_right">
-    <selfCollide>true</selfCollide>
-    <mu1 value="0.09"/>
-    <mu2 value="0.09"/>
-    <kp value="10000000.0" />
-    <kd value="10000" />
-    <fdir1 value="0 0 0"/>
-  </gazebo>
-  <link name="wheel_front_right">
-    <inertial>
-      <mass value="0.01"/>
-      <origin rpy="0 0 0" xyz="0 0 0"/>
-      <inertia ixx="1" ixy="0.0" ixz="0.0" iyy="1" iyz="0.0" izz="1"/>
-    </inertial>
-    <collision name="wheel_front_right_collision">
-      <origin rpy="0 0 0" xyz="0 0 0"/>
-      <geometry>
-        <mesh filename="package://robot_description/models/laser_robot/omni_wheel/meshes/roda_omni.obj" scale="1 1 1"/>
-      </geometry>
-    </collision>
-    <visual name="wheel_front_right_visual">
-      <origin rpy="0 0 0" xyz="0 0 0"/>
-      <geometry>
-        <mesh filename="package://robot_description/models/laser_robot/omni_wheel/meshes/roda_omni.obj" scale="1 1 1"/>
-      </geometry>
-    </visual>
-  </link>
-  <gazebo reference="wheel_rear_right">
-    <selfCollide>true</selfCollide>
-    <mu1 value="0.09"/>
-    <mu2 value="0.09"/>
-    <kp value="10000000.0" />
-    <kd value="10000" />
-    <fdir1 value="0 0 0"/>
-  </gazebo>
-  <link name="wheel_rear_right">
-    <inertial>
-      <mass value="0.01"/>
-      <origin rpy="0 0 0" xyz="0 0 0"/>
-      <inertia ixx="1" ixy="0.0" ixz="0.0" iyy="1" iyz="0.0" izz="1"/>
-    </inertial>
-    <collision name="wheel_rear_right_collision">
-      <origin rpy="0 0 0" xyz="0 0 0"/>
-      <geometry>
-        <mesh filename="package://robot_description/models/laser_robot/omni_wheel/meshes/roda_omni.obj" scale="1 1 1"/>
-      </geometry>
-    </collision>
-    <visual name="wheel_rear_right_visual">
-      <origin rpy="0 0 0" xyz="0 0 0"/>
-      <geometry>
-        <mesh filename="package://robot_description/models/laser_robot/omni_wheel/meshes/roda_omni.obj" scale="1 1 1"/>
-      </geometry>
-    </visual>
-  </link>
-  <gazebo reference="wheel_front_left">
-    <selfCollide>true</selfCollide>
-    <mu1 value="0.09"/>
-    <mu2 value="0.09"/>
-    <kp value="10000000.0" />
-    <kd value="10000" />
-    <fdir1 value="0 0 0"/>
-  </gazebo>
-  <link name="wheel_front_left">
-    <inertial>
-      <mass value="0.01"/>
-      <origin rpy="0 0 0" xyz="0 0 0"/>
-      <inertia ixx="1" ixy="0.0" ixz="0.0" iyy="1" iyz="0.0" izz="1"/>
-    </inertial>
-    <collision name="wheel_front_left_collision">
-      <origin rpy="0 0 0" xyz="0 0 0"/>
-      <geometry>
-        <mesh filename="package://robot_description/models/laser_robot/omni_wheel/meshes/roda_omni.obj" scale="1 1 1"/>
-      </geometry>
-    </collision>
-    <visual name="wheel_front_left_visual">
-      <origin rpy="0 0 0" xyz="0 0 0"/>
-      <geometry>
-        <mesh filename="package://robot_description/models/laser_robot/omni_wheel/meshes/roda_omni.obj" scale="1 1 1"/>
-      </geometry>
-    </visual>
-  </link>
-  <gazebo reference="wheel_rear_left">
-    <selfCollide>true</selfCollide>
-    <mu1 value="0.09"/>
-    <mu2 value="0.09"/>
-    <kp value="10000000.0" />
-    <kd value="10000" />
-    <fdir1 value="0 0 0"/>
-  </gazebo>
-  <link name="wheel_rear_left">
-    <inertial>
-      <mass value="0.01"/>
-      <origin rpy="0 0 0" xyz="0 0 0"/>
-      <inertia ixx="1" ixy="0.0" ixz="0.0" iyy="1" iyz="0.0" izz="1"/>
-    </inertial>
-    <collision name="wheel_rear_left_collision">
-      <origin rpy="0 0 0" xyz="0 0 0"/>
-      <geometry>
-        <mesh filename="package://robot_description/models/laser_robot/omni_wheel/meshes/roda_omni.obj" scale="1 1 1"/>
-      </geometry>
-    </collision>
-    <visual name="wheel_rear_left_visual">
-      <origin rpy="0 0 0" xyz="0 0 0"/>
-      <geometry>
-        <mesh filename="package://robot_description/models/laser_robot/omni_wheel/meshes/roda_omni.obj" scale="1 1 1"/>
-      </geometry>
-    </visual>
-  </link>
-  <gazebo reference="piston">
-    <selfCollide>false</selfCollide>
-    <mu1 value="0.1"/>
-    <mu2 value="0.1"/>
-    <kp value="10000000.0" />
-    <kd value="10000" />
-    <fdir1 value="0 0 0"/>
-  </gazebo>
-  <link name="piston">
-    <inertial>
-      <mass value="0.3"/>
-      <origin rpy="0  0  0" xyz="0 0 0"/>
-      <inertia ixx="0" ixy="0" ixz="0" iyy="0" iyz="0" izz="0"/>
-    </inertial>
-    <collision name="piston_collision">
-      <origin rpy="0  0  0" xyz="0 0 0"/>
-      <geometry>
-        <mesh filename="package://robot_description/models/laser_robot/meshes/piston.dae" scale="1 1 1"/>
-      </geometry>
-    </collision>
-    <visual name="piston_visual">
-      <origin rpy="0  0  0" xyz="0 0 0"/>
-      <geometry>
-        <mesh filename="package://robot_description/models/laser_robot/meshes/piston.dae" scale="1 1 1"/>
-      </geometry>
-    </visual>
-  </link>
-  <gazebo reference="tray">
-    <selfCollide>false</selfCollide>
-    <mu1 value="0.1"/>
-    <mu2 value="0.1"/>
-    <kp value="10000000.0" />
-    <kd value="10000" />
-    <fdir1 value="0 0 0"/>
-  </gazebo>
-  <link name="tray">
-    <inertial>
-      <mass value="0.5"/>
-      <origin rpy="0 0 0" xyz="0 0 0"/>
-      <inertia ixx="0" ixy="0.0" ixz="0.0" iyy="0" iyz="0.0" izz="0"/>
-    </inertial>
-    <collision name="tray_collision">
-      <origin rpy="0 0 0" xyz="0 0 0"/>
-      <geometry>
-        <mesh filename="package://robot_description/models/laser_robot/meshes/tray.dae" scale="1 1 1"/>
-      </geometry>
-    </collision>
-    <visual name="tray_visual">
-      <origin rpy="0 0 0" xyz="0 0 0"/>
-      <geometry>
-        <mesh filename="package://robot_description/models/laser_robot/meshes/tray.dae" scale="1 1 1"/>
-      </geometry>
-    </visual>
-  </link>
-  <link name="camera_1">
-    <inertial>
-      <mass value="0.1"/>
-      <origin rpy="0 0 0" xyz="0 0 0"/>
-      <inertia ixx="1" ixy="0" ixz="0" iyy="1" iyz="0" izz="1"/>
-    </inertial>
-    <collision name="camera_1_collision">
-      <origin rpy="0 0 0" xyz="0 0 0"/>
-      <geometry>
-        <mesh filename="package://robot_description/models/laser_robot/camera/meshes/camera.obj" scale="0.5 0.5 0.5"/>
-      </geometry>
-    </collision>
-    <visual name="camera_1_visual">
-      <origin rpy="0 0 1.57" xyz="0 0 0"/>
-      <geometry>
-        <mesh filename="package://robot_description/models/laser_robot/camera/meshes/camera.obj" scale="0.5 0.5 0.5"/>
-      </geometry>
-    </visual>
-  </link>
-  <gazebo reference="right_wheel">
-    <selfCollide>false</selfCollide>
-    <mu1 value="100"/>
-    <mu2 value="50"/>
-    <kp value="10000000.0" />
-    <kd value="1000" />
-    <fdir1 value="0 0 0"/>
-  </gazebo>
-  <link name="right_wheel">
-    <inertial>
-      <mass value="1"/>
-      <origin rpy="0 0 0" xyz="0 0 0"/>
-      <inertia ixx="1" ixy="0" ixz="0" iyy="1" iyz="0" izz="1"/>
-    </inertial>
-    <collision name="right_wheel_collision">
-      <origin rpy="0 0 0" xyz="0 0 0"/>
-      <geometry>
-        <mesh filename="package://robot_description/models/laser_robot/wheel/meshes/roda.obj" scale="1 1 1"/>
-      </geometry>
-    </collision>
-    <visual name="right_wheel_visual">
-      <origin rpy="0 0 0" xyz="0 0 0"/>
-      <geometry>
-        <mesh filename="package://robot_description/models/laser_robot/wheel/meshes/roda.obj" scale="1 1 1"/>
-      </geometry>
-    </visual>
-  </link>
-  <gazebo reference="left_wheel">
-    <selfCollide>false</selfCollide>
-    <mu1 value="100"/>
-    <mu2 value="50"/>
-    <kp value="10000000.0" />
-    <kd value="1000" />
-    <fdir1 value="0 0 0"/>
-  </gazebo>
-  <link name="left_wheel">
-    <inertial>
-      <mass value="1"/>
-      <origin rpy="0 0 0" xyz="0 0 0"/>
-      <inertia ixx="1" ixy="0" ixz="0" iyy="1" iyz="0" izz="1"/>
-    </inertial>
-    <collision name="left_wheel_collision">
-      <origin rpy="0 0 0" xyz="0 0 0"/>
-      <geometry>
-        <mesh filename="package://robot_description/models/laser_robot/wheel/meshes/roda.obj" scale="1 1 1"/>
-      </geometry>
-    </collision>
-    <visual name="left_wheel_visual">
-      <origin rpy="0 0 0" xyz="0 0 0"/>
-      <geometry>
-        <mesh filename="package://robot_description/models/laser_robot/wheel/meshes/roda.obj" scale="1 1 1"/>
-      </geometry>
-    </visual>
-  </link>
-  <link name="lidar">
-    <inertial>
-      <mass value="0.1"/>
-      <origin rpy="0 0 0" xyz="0 0 0"/>
-      <inertia ixx="1" ixy="0" ixz="0" iyy="1" iyz="0" izz="1"/>
-    </inertial>
-    <collision name="lidar_collision">
-      <origin rpy="0 0 0" xyz="0 0 0"/>
-      <geometry>
-        <mesh filename="package://robot_description/models/laser_robot/lidar/meshes/lidar.obj" scale="0.5 0.5 0.5"/>
-      </geometry>
-    </collision>
-    <visual name="lidar_visual">
-      <origin rpy="0 1.57 1.57" xyz="0 0 0"/>
-      <geometry>
-        <mesh filename="package://robot_description/models/laser_robot/lidar/meshes/lidar.obj" scale="0.5 0.5 0.5"/>
-      </geometry>
-    </visual>
-  </link>
-  <link name="rplidar">
-    <inertial>
-      <mass value="0.1"/>
-      <origin rpy="0 0 0" xyz="0 0 0"/>
-      <inertia ixx="1" ixy="0" ixz="0" iyy="1" iyz="0" izz="1"/>
-    </inertial>
-    <collision name="rplidar_collision">
-      <origin rpy="0 0 1.20" xyz="-0.03 0.02 -0.02"/>
-      <geometry>
-        <mesh filename="package://robot_description/models/laser_robot/meshes/rplidar.dae" scale="0.7 0.7 0.7"/>
-      </geometry>
-    </collision>
-    <visual name="rplidar_visual">
-      <origin rpy="0 0 1.20" xyz="-0.03 0.02 -0.02"/>
-      <geometry>
-        <mesh filename="package://robot_description/models/laser_robot/meshes/rplidar.dae" scale="0.7 0.7 0.7"/>
-      </geometry>
-    </visual>
-  </link>
+  <!--=========================== ROBOT PARTS ===========================-->
+  <xacro:include filename="$(find robot_description)/urdf/robot_parts/carcaca.xacro" />
+  <xacro:include filename="$(find robot_description)/urdf/robot_parts/right_wheel.xacro" />
+  <xacro:include filename="$(find robot_description)/urdf/robot_parts/left_wheel.xacro" />
+  <xacro:include filename="$(find robot_description)/urdf/robot_parts/tray.xacro" />
+  <xacro:include filename="$(find robot_description)/urdf/robot_parts/piston.xacro" />
+  <xacro:include filename="$(find robot_description)/urdf/robot_parts/left_rear_wheel.xacro" />
+  <xacro:include filename="$(find robot_description)/urdf/robot_parts/right_rear_wheel.xacro" />
+  <xacro:include filename="$(find robot_description)/urdf/robot_parts/left_front_wheel.xacro" />
+  <xacro:include filename="$(find robot_description)/urdf/robot_parts/right_front_wheel.xacro" />
+  <!--=========================== SENSORS ===========================-->
+  <xacro:arg name="sensor_imu" default="false" />
+  <xacro:arg name="sensor_lidar" default="false" />
+  <xacro:arg name="sensor_rplidar" default="false" />
+  <xacro:arg name="sensor_camera" default="false" />
+  <xacro:if value="$(arg sensor_imu)">
+    <xacro:include filename="$(find robot_description)/urdf/sensors/imu.xacro" />
+  </xacro:if>
+  <xacro:if value="$(arg sensor_lidar)">
+    <xacro:include filename="$(find robot_description)/urdf/sensors/lidar.xacro" />
+  </xacro:if>
+  <xacro:if value="$(arg sensor_rplidar)">
+    <xacro:include filename="$(find robot_description)/urdf/sensors/rplidar.xacro" />
+  </xacro:if>
+  <xacro:if value="$(arg sensor_camera)">
+    <xacro:include filename="$(find robot_description)/urdf/sensors/camera.xacro" />
+  </xacro:if>
 </robot>
