Commit message: Adding macros

File: robot_description/urdf/robot.urdf.xacro (robot description, xacro)
@@ -5,12 +5,8 @@
   <!--=========================== ROBOT PARTS ===========================-->
   <xacro:include filename="$(find robot_description)/urdf/robot_parts/carcaca.xacro" />
-  <xacro:include filename="$(find robot_description)/urdf/robot_parts/right_wheel.xacro" />
-  <xacro:include filename="$(find robot_description)/urdf/robot_parts/left_wheel.xacro" />
+  <xacro:include filename="$(find robot_description)/urdf/robot_parts/traction_wheel.xacro" />
   <xacro:include filename="$(find robot_description)/urdf/robot_parts/tray.xacro" />
   <xacro:include filename="$(find robot_description)/urdf/robot_parts/piston.xacro" />
-  <xacro:include filename="$(find robot_description)/urdf/robot_parts/left_rear_wheel.xacro" />
-  <xacro:include filename="$(find robot_description)/urdf/robot_parts/right_rear_wheel.xacro" />
-  <xacro:include filename="$(find robot_description)/urdf/robot_parts/left_front_wheel.xacro" />
-  <xacro:include filename="$(find robot_description)/urdf/robot_parts/right_front_wheel.xacro" />
+  <xacro:include filename="$(find robot_description)/urdf/robot_parts/omni_wheel.xacro" />
   <!--=========================== SENSORS ===========================-->
   <xacro:arg name="sensor_imu" default="false" />

File: robot_description/urdf/robot_parts/carcaca.xacro (robot description, xacro)
@@ -1,30 +1,33 @@
 <?xml version="1.0"?>
 <robot xmlns:xacro="http://www.ros.org/wiki/xacro">
-    <gazebo reference="carcaca">
-        <selfCollide>true</selfCollide>
-        <mu1 value="0.3" />
-        <mu2 value="0.3" />
-        <kp value="10000000.0" />
-        <kd value="1000" />
-        <fdir1 value="0 0 0" />
-    </gazebo>
-    <link name="carcaca">
-        <inertial>
-            <mass value="15" />
-            <origin rpy="0  0  3.14" xyz="0  0  0.0118" />
-            <inertia ixx="1" ixy="0" ixz="0" iyy="1" iyz="0" izz="1" />
-        </inertial>
-        <collision name="carcaca_collision">
-            <origin rpy="0  0  3.14" xyz="0  0  0.0118" />
-            <geometry>
-                <mesh filename="package://robot_description/models/laser_robot/meshes/carcaca.dae" scale="1 1 1" />
-            </geometry>
-        </collision>
-        <visual name="carcaca_visual">
-            <origin rpy="0  0  3.14" xyz="0  0  0.0118" />
-            <geometry>
-                <mesh filename="package://robot_description/models/laser_robot/meshes/carcaca.dae" scale="1 1 1" />
-            </geometry>
-        </visual>
-    </link>
+    <xacro:macro name="base" params="base_link">
+        <gazebo reference="${base_link}">
+            <selfCollide>true</selfCollide>
+            <mu1 value="0.3" />
+            <mu2 value="0.3" />
+            <kp value="10000000.0" />
+            <kd value="1000" />
+            <fdir1 value="0 0 0" />
+        </gazebo>
+        <link name="${base_link}">
+            <inertial>
+                <mass value="15" />
+                <origin rpy="0  0  3.14" xyz="0  0  0.0118" />
+                <inertia ixx="1" ixy="0" ixz="0" iyy="1" iyz="0" izz="1" />
+            </inertial>
+            <collision name="${base_link}_collision">
+                <origin rpy="0  0  3.14" xyz="0  0  0.0118" />
+                <geometry>
+                    <mesh filename="package://robot_description/models/laser_robot/meshes/carcaca.dae" scale="1 1 1" />
+                </geometry>
+            </collision>
+            <visual name="${base_link}_visual">
+                <origin rpy="0  0  3.14" xyz="0  0  0.0118" />
+                <geometry>
+                    <mesh filename="package://robot_description/models/laser_robot/meshes/carcaca.dae" scale="1 1 1" />
+                </geometry>
+            </visual>
+        </link>
+    </xacro:macro>
+    <xacro:base base_link="carcaca" />
 </robot>

File: robot_description/urdf/robot_parts/piston.xacro (robot description, xacro)
@@ -1,37 +1,40 @@
 <?xml version="1.0"?>
 <robot xmlns:xacro="http://www.ros.org/wiki/xacro">
-    <joint name="joint_piston" type="prismatic">
-        <parent link="carcaca" />
-        <child link="piston" />
-        <origin rpy="0 0 0" xyz="0 0 0.1318" />
-        <axis xyz="0 0 1" />
-        <limit effort="0" lower="0" upper="0.04" velocity="0" />
-    </joint>
-    <gazebo reference="piston">
-        <selfCollide>false</selfCollide>
-        <mu1 value="0.1" />
-        <mu2 value="0.1" />
-        <kp value="10000000.0" />
-        <kd value="10000" />
-        <fdir1 value="0 0 0" />
-    </gazebo>
-    <link name="piston">
-        <inertial>
-            <mass value="0.3" />
-            <origin rpy="0  0  0" xyz="0 0 0" />
-            <inertia ixx="0" ixy="0" ixz="0" iyy="0" iyz="0" izz="0" />
-        </inertial>
-        <collision name="piston_collision">
-            <origin rpy="0  0  0" xyz="0 0 0" />
-            <geometry>
-                <mesh filename="package://robot_description/models/laser_robot/meshes/piston.dae" scale="1 1 1" />
-            </geometry>
-        </collision>
-        <visual name="piston_visual">
-            <origin rpy="0  0  0" xyz="0 0 0" />
-            <geometry>
-                <mesh filename="package://robot_description/models/laser_robot/meshes/piston.dae" scale="1 1 1" />
-            </geometry>
-        </visual>
-    </link>
+    <xacro:macro name="piston" params="prefix">
+        <joint name="joint_${prefix}" type="prismatic">
+            <parent link="carcaca" />
+            <child link="${prefix}" />
+            <origin rpy="0 0 0" xyz="0 0 0.1318" />
+            <axis xyz="0 0 1" />
+            <limit effort="0" lower="0" upper="0.04" velocity="0" />
+        </joint>
+        <gazebo reference="${prefix}">
+            <selfCollide>false</selfCollide>
+            <mu1 value="0.1" />
+            <mu2 value="0.1" />
+            <kp value="10000000.0" />
+            <kd value="10000" />
+            <fdir1 value="0 0 0" />
+        </gazebo>
+        <link name="${prefix}">
+            <inertial>
+                <mass value="0.3" />
+                <origin rpy="0  0  0" xyz="0 0 0" />
+                <inertia ixx="0" ixy="0" ixz="0" iyy="0" iyz="0" izz="0" />
+            </inertial>
+            <collision name="${prefix}_collision">
+                <origin rpy="0  0  0" xyz="0 0 0" />
+                <geometry>
+                    <mesh filename="package://robot_description/models/laser_robot/meshes/piston.dae" scale="1 1 1" />
+                </geometry>
+            </collision>
+            <visual name="${prefix}_visual">
+                <origin rpy="0  0  0" xyz="0 0 0" />
+                <geometry>
+                    <mesh filename="package://robot_description/models/laser_robot/meshes/piston.dae" scale="1 1 1" />
+                </geometry>
+            </visual>
+        </link>
+    </xacro:macro>
+    <xacro:piston prefix="piston" />
 </robot>

File: robot_description/urdf/robot_parts/tray.xacro (robot description, xacro)
@@ -1,36 +1,39 @@
 <?xml version="1.0"?>
 <robot xmlns:xacro="http://www.ros.org/wiki/xacro">
-    <joint name="joint_tray" type="continuous">
-        <parent link="piston" />
-        <child link="tray" />
-        <origin rpy="0 0 0" xyz="0 0 0" />
-        <axis xyz="0 0 1" />
-    </joint>
-    <gazebo reference="tray">
-        <selfCollide>false</selfCollide>
-        <mu1 value="0.1" />
-        <mu2 value="0.1" />
-        <kp value="10000000.0" />
-        <kd value="10000" />
-        <fdir1 value="0 0 0" />
-    </gazebo>
-    <link name="tray">
-        <inertial>
-            <mass value="0.5" />
+    <xacro:macro name="tray" params="prefix">
+        <joint name="joint_${prefix}" type="continuous">
+            <parent link="piston" />
+            <child link="${prefix}" />
             <origin rpy="0 0 0" xyz="0 0 0" />
-            <inertia ixx="0" ixy="0.0" ixz="0.0" iyy="0" iyz="0.0" izz="0" />
-        </inertial>
-        <collision name="tray_collision">
-            <origin rpy="0 0 0" xyz="0 0 0" />
-            <geometry>
-                <mesh filename="package://robot_description/models/laser_robot/meshes/tray.dae" scale="1 1 1" />
-            </geometry>
-        </collision>
-        <visual name="tray_visual">
-            <origin rpy="0 0 0" xyz="0 0 0" />
-            <geometry>
-                <mesh filename="package://robot_description/models/laser_robot/meshes/tray.dae" scale="1 1 1" />
-            </geometry>
-        </visual>
-    </link>
+            <axis xyz="0 0 1" />
+        </joint>
+        <gazebo reference="${prefix}">
+            <selfCollide>false</selfCollide>
+            <mu1 value="0.1" />
+            <mu2 value="0.1" />
+            <kp value="10000000.0" />
+            <kd value="10000" />
+            <fdir1 value="0 0 0" />
+        </gazebo>
+        <link name="${prefix}">
+            <inertial>
+                <mass value="0.5" />
+                <origin rpy="0 0 0" xyz="0 0 0" />
+                <inertia ixx="0" ixy="0.0" ixz="0.0" iyy="0" iyz="0.0" izz="0" />
+            </inertial>
+            <collision name="${prefix}_collision">
+                <origin rpy="0 0 0" xyz="0 0 0" />
+                <geometry>
+                    <mesh filename="package://robot_description/models/laser_robot/meshes/tray.dae" scale="1 1 1" />
+                </geometry>
+            </collision>
+            <visual name="${prefix}_visual">
+                <origin rpy="0 0 0" xyz="0 0 0" />
+                <geometry>
+                    <mesh filename="package://robot_description/models/laser_robot/meshes/tray.dae" scale="1 1 1" />
+                </geometry>
+            </visual>
+        </link>
+    </xacro:macro>
+    <xacro:tray prefix="tray" />
 </robot>

Commit message: fixed issues in rviz

File: robot_description/urdf/robot.urdf.xacro (robot description, xacro)
@@ -10,8 +10,8 @@
   <xacro:include filename="$(find robot_description)/urdf/robot_parts/omni_wheel.xacro" />
   <!--=========================== SENSORS ===========================-->
-  <xacro:arg name="sensor_imu" default="false" />
-  <xacro:arg name="sensor_lidar" default="false" />
-  <xacro:arg name="sensor_rplidar" default="false" />
-  <xacro:arg name="sensor_camera" default="false" />
+  <xacro:arg name="sensor_imu" default="true" />
+  <xacro:arg name="sensor_lidar" default="true" />
+  <xacro:arg name="sensor_rplidar" default="true" />
+  <xacro:arg name="sensor_camera" default="true" />
   <xacro:if value="$(arg sensor_imu)">
     <xacro:include filename="$(find robot_description)/urdf/sensors/imu.xacro" />

File: robot_description/urdf/robot_parts/piston.xacro (robot description, xacro)
@@ -5,4 +5,5 @@
             <parent link="carcaca" />
             <child link="${prefix}" />
+            <!-- <dynamics friction="5.0" /> -->
             <origin rpy="0 0 0" xyz="0 0 0.1318" />
             <axis xyz="0 0 1" />
@@ -10,5 +11,5 @@
         </joint>
         <gazebo reference="${prefix}">
-            <selfCollide>false</selfCollide>
+            <selfCollide>true</selfCollide>
             <mu1 value="0.1" />
             <mu2 value="0.1" />

File: robot_description/urdf/robot_parts/tray.xacro (robot description, xacro)
@@ -5,9 +5,10 @@
             <parent link="piston" />
             <child link="${prefix}" />
+            <!-- <dynamics friction="5.0" /> -->
             <origin rpy="0 0 0" xyz="0 0 0" />
             <axis xyz="0 0 1" />
         </joint>
         <gazebo reference="${prefix}">
-            <selfCollide>false</selfCollide>
+            <selfCollide>true</selfCollide>
             <mu1 value="0.1" />
             <mu2 value="0.1" />

File: robot_description/urdf/sensors/lidar.xacro (robot description, xacro)
@@ -1,62 +1,62 @@
 <?xml version="1.0"?>
 <robot xmlns:xacro="http://www.ros.org/wiki/xacro">
-    <gazebo reference="lidar">
-        <sensor type="ray" name="laser_sensor">
-          <pose>0 0 0 0 0 0</pose>
-          <visualize>false</visualize>
-          <update_rate>20</update_rate>
-          <ray>
-            <scan>
-              <horizontal>
-                <samples>${14400/20}</samples>
-                <resolution>1</resolution>
-                <min_angle>-1.1781</min_angle>
-                <max_angle>1.1781</max_angle>
-              </horizontal>
-            </scan>
-            <range>
-              <min>0.15</min>
-              <max>14.0</max>
-              <resolution>0.01</resolution>
-            </range>
-            <noise>
-              <type>gaussian</type>
-              <!-- Noise parameters based on published spec for Hokuyo laser
+  <gazebo reference="lidar">
+    <sensor type="ray" name="laser_sensor">
+      <pose>0 0 0 0 0 0</pose>
+      <visualize>false</visualize>
+      <update_rate>20</update_rate>
+      <ray>
+        <scan>
+          <horizontal>
+            <samples>${14400/20}</samples>
+            <resolution>1</resolution>
+            <min_angle>-1.1781</min_angle>
+            <max_angle>1.1781</max_angle>
+          </horizontal>
+        </scan>
+        <range>
+          <min>0.15</min>
+          <max>14.0</max>
+          <resolution>0.01</resolution>
+        </range>
+        <noise>
+          <type>gaussian</type>
+          <!-- Noise parameters based on published spec for Hokuyo laser
                    achieving "+-30mm" accuracy at range < 10m.  A mean of 0.0m and
                    stddev of 0.01m will put 99.7% of samples within 0.03m of the true
                    reading. -->
-              <mean>0.0</mean>
-              <stddev>0.01</stddev>
-            </noise>
-          </ray>
-          <plugin name="gazebo_ros_head_hokuyo_controller" filename="libgazebo_ros_laser.so">
-            <topicName>/my_robot/laser/scan</topicName>
-            <frameName>lidar</frameName>
-          </plugin>
-        </sensor>
-      </gazebo>
-      <joint name="joint_lidar" type="fixed">
-        <parent link="carcaca" />
-        <child link="lidar" />
-        <origin rpy="0 0 -1.57" xyz="-0.0005 -0.23 0.109" />
-      </joint>
-      <link name="lidar">
-        <inertial>
-          <mass value="0.1" />
-          <origin rpy="0 0 0" xyz="0 0 0" />
-          <inertia ixx="1" ixy="0" ixz="0" iyy="1" iyz="0" izz="1" />
-        </inertial>
-        <collision name="lidar_collision">
-          <origin rpy="0 0 0" xyz="0 0 0" />
-          <geometry>
-            <mesh filename="package://robot_description/models/laser_robot/lidar/meshes/lidar.obj" scale="0.5 0.5 0.5" />
-          </geometry>
-        </collision>
-        <visual name="lidar_visual">
-          <origin rpy="0 1.57 1.57" xyz="0 0 0" />
-          <geometry>
-            <mesh filename="package://robot_description/models/laser_robot/lidar/meshes/lidar.obj" scale="0.5 0.5 0.5" />
-          </geometry>
-        </visual>
-      </link>
+          <mean>0.0</mean>
+          <stddev>0.01</stddev>
+        </noise>
+      </ray>
+      <plugin name="gazebo_ros_head_hokuyo_controller" filename="libgazebo_ros_laser.so">
+        <topicName>/my_robot/laser/scan</topicName>
+        <frameName>lidar</frameName>
+      </plugin>
+    </sensor>
+  </gazebo>
+  <joint name="joint_lidar" type="fixed">
+    <parent link="carcaca" />
+    <child link="lidar" />
+    <origin rpy="0 0 -1.57" xyz="-0.0005 -0.23 0.109" />
+  </joint>
+  <link name="lidar">
+    <inertial>
+      <mass value="0.1" />
+      <origin rpy="0 0 0" xyz="0 0 0" />
+      <inertia ixx="1" ixy="0" ixz="0" iyy="1" iyz="0" izz="1" />
+    </inertial>
+    <collision name="lidar_collision">
+      <origin rpy="0 0 0" xyz="0 0 0" />
+      <geometry>
+        <mesh filename="package://robot_description/models/laser_robot/lidar/meshes/lidar.obj" scale="0.5 0.5 0.5" />
+      </geometry>
+    </collision>
+    <visual name="lidar_visual">
+      <origin rpy="0 1.57 1.57" xyz="0 0 0" />
+      <geometry>
+        <mesh filename="package://robot_description/models/laser_robot/lidar/meshes/lidar.obj" scale="0.5 0.5 0.5" />
+      </geometry>
+    </visual>
+  </link>
 </robot>

File: robot_description/urdf/sensors/rplidar.xacro (robot description, xacro)
@@ -1,62 +1,62 @@
 <?xml version="1.0"?>
 <robot xmlns:xacro="http://www.ros.org/wiki/xacro">
-    <gazebo reference="rplidar">
-        <sensor type="ray" name="laser_sensor">
-          <pose>0 0 0 0 0 0</pose>
-          <visualize>false</visualize>
-          <update_rate>20</update_rate>
-          <ray>
-            <scan>
-              <horizontal>
-                <samples>${14400/20}</samples>
-                <resolution>1</resolution>
-                <min_angle>-3.14159265359</min_angle>
-                <max_angle>3.14159265359</max_angle>
-              </horizontal>
-            </scan>
-            <range>
-              <min>0.15</min>
-              <max>14.0</max>
-              <resolution>0.01</resolution>
-            </range>
-            <noise>
-              <type>gaussian</type>
-              <!-- Noise parameters based on published spec for Hokuyo laser
+  <gazebo reference="rplidar">
+    <sensor type="ray" name="laser_sensor">
+      <pose>0 0 0 0 0 0</pose>
+      <visualize>false</visualize>
+      <update_rate>20</update_rate>
+      <ray>
+        <scan>
+          <horizontal>
+            <samples>${14400/20}</samples>
+            <resolution>1</resolution>
+            <min_angle>-3.14159265359</min_angle>
+            <max_angle>3.14159265359</max_angle>
+          </horizontal>
+        </scan>
+        <range>
+          <min>0.15</min>
+          <max>14.0</max>
+          <resolution>0.01</resolution>
+        </range>
+        <noise>
+          <type>gaussian</type>
+          <!-- Noise parameters based on published spec for Hokuyo laser
                    achieving "+-30mm" accuracy at range < 10m.  A mean of 0.0m and
                    stddev of 0.01m will put 99.7% of samples within 0.03m of the true
                    reading. -->
-              <mean>0.0</mean>
-              <stddev>0.01</stddev>
-            </noise>
-          </ray>
-          <plugin name="gazebo_ros_head_hokuyo_controller" filename="libgazebo_ros_laser.so">
-            <topicName>/my_robot/rplidar/laser/scan</topicName>
-            <frameName>rplidar</frameName>
-          </plugin>
-        </sensor>
-      </gazebo>
-      <joint name="joint_rplidar" type="fixed">
-        <parent link="carcaca" />
-        <child link="rplidar" />
-        <origin rpy="0 0 0" xyz="0.14 -0.17 0.27" />
-      </joint>
-      <link name="rplidar">
-        <inertial>
-          <mass value="0.1" />
-          <origin rpy="0 0 0" xyz="0 0 0" />
-          <inertia ixx="1" ixy="0" ixz="0" iyy="1" iyz="0" izz="1" />
-        </inertial>
-        <collision name="rplidar_collision">
-          <origin rpy="0 0 1.20" xyz="-0.03 0.02 -0.02" />
-          <geometry>
-            <mesh filename="package://robot_description/models/laser_robot/meshes/rplidar.dae" scale="0.7 0.7 0.7" />
-          </geometry>
-        </collision>
-        <visual name="rplidar_visual">
-          <origin rpy="0 0 1.20" xyz="-0.03 0.02 -0.02" />
-          <geometry>
-            <mesh filename="package://robot_description/models/laser_robot/meshes/rplidar.dae" scale="0.7 0.7 0.7" />
-          </geometry>
-        </visual>
-      </link>
+          <mean>0.0</mean>
+          <stddev>0.01</stddev>
+        </noise>
+      </ray>
+      <plugin name="gazebo_ros_head_hokuyo_controller" filename="libgazebo_ros_laser.so">
+        <topicName>/my_robot/rplidar/laser/scan</topicName>
+        <frameName>rplidar</frameName>
+      </plugin>
+    </sensor>
+  </gazebo>
+  <joint name="joint_rplidar" type="fixed">
+    <parent link="carcaca" />
+    <child link="rplidar" />
+    <origin rpy="0 0 0" xyz="0.14 -0.17 0.27" />
+  </joint>
+  <link name="rplidar">
+    <inertial>
+      <mass value="0.1" />
+      <origin rpy="0 0 0" xyz="0 0 0" />
+      <inertia ixx="1" ixy="0" ixz="0" iyy="1" iyz="0" izz="1" />
+    </inertial>
+    <collision name="rplidar_collision">
+      <origin rpy="0 0 1.20" xyz="-0.03 0.02 -0.02" />
+      <geometry>
+        <mesh filename="package://robot_description/models/laser_robot/meshes/rplidar.dae" scale="0.7 0.7 0.7" />
+      </geometry>
+    </collision>
+    <visual name="rplidar_visual">
+      <origin rpy="0 0 1.20" xyz="-0.03 0.02 -0.02" />
+      <geometry>
+        <mesh filename="package://robot_description/models/laser_robot/meshes/rplidar.dae" scale="0.7 0.7 0.7" />
+      </geometry>
+    </visual>
+  </link>
 </robot>
