Commit message: AprilTag

File: robot_description/urdf/sensors/camera.xacro (robot description, xacro)
@@ -42,5 +42,5 @@
         <parent link="carcaca" />
         <child link="camera_1" />
-        <origin rpy="0 1.57 0" xyz="0 -0.127 0.0367" />
+        <origin rpy="0 1.57 0" xyz="0 0 0.0367" />
     </joint>
     <link name="camera_1">
